File: pcb/CSPS.kicad_sch (KiCad schematic)
At the start: 43 parts, among them J1 Conn_02x32_Counter_Clockwise, J10 Conn_01x02, J11 Conn_01x02, J12 Conn_01x06, J13 Conn_01x06, J2 Conn_01x02, J3 Conn_01x03, J4 XT30, J5 XT30, J6 XT30, J7 XT30, J8 Conn_01x04, J9 Conn_01x02, Q1 AO3400A, Q2 AO3400A, SW1 SW_Push, U1 CH32V003AxMx, U2 TLV70433DBVR

Commit message: PCB Update
Parts:
- C1, C3, C5, C6, C7: LCSC C126469 -> C24497
- C2: LCSC C98192 -> C29823
- C4: LCSC C19110 -> C50254
- D2: LCSC C965815 -> C3646937
- R1, R2: LCSC C114237 -> C17948
- R10, R13, R8: LCSC C2907294 -> C17901
- R11: LCSC C2907329 -> C4502
- R12, R3, R5, R9: LCSC C2907423 -> C17902
- R4: LCSC C2907295 -> C4410
- R6: value 22K -> 15K; LCSC C2907309 -> C25828
- R7: LCSC C105427 -> C17936
Other:
- moved on the sheet: D3, R6
